Commit message: Add arm namespace to camera

File: robots/z1_description/xacro/z1.xacro (robot description, xacro)
@@ -306,5 +306,5 @@
             </gazebo>
             <xacro:if value="${realsense}">
-                <xacro:z1_realsense_wrist_mount />
+                <xacro:z1_realsense_wrist_mount robot_namespace="${robot_namespace}" sim="${sim}" />
             </xacro:if>
         </xacro:if>
@@ -385,5 +385,6 @@
                 <!-- add RealSense D435i (the mesh is actually the non-IMU version) -->
                 <xacro:include filename="$(find realsense2_description)/urdf/_d435i.urdf.xacro" />
-                <xacro:sensor_d435i name="wrist_camera" parent="robotiq_arg2f_base_link"
+                <xacro:sensor_d435i name="${robot_namespace}/wrist_camera"
+                    parent="robotiq_arg2f_base_link"
                     use_nominal_extrinsics="${sim}">
                     <!-- XYZ NEEDS TUNING -->
@@ -392,5 +393,5 @@
                 <!-- Simulated Realsense -->
                 <xacro:include filename="$(find z1_description)/xacro/realsense_d435.gazebo" />
-                <xacro:realsense_d435_gazebo name="wrist_camera">
+                <xacro:realsense_d435_gazebo name="${robot_namespace}/wrist_camera">
                     <origin xyz="0 0 0" rpy="0 0 0" />
                 </xacro:realsense_d435_gazebo>

File: robots/z1_description/xacro/z1_realsense_wrist_mount.xacro (robot description, xacro)
@@ -16,5 +16,5 @@
     xmlns:physics="http://playerstage.sourceforge.net/gazebo/xmlschema/#physics"
     xmlns:xacro="http://www.ros.org/wiki/xacro">
-    <xacro:macro name="z1_realsense_wrist_mount">
+    <xacro:macro name="z1_realsense_wrist_mount" params="robot_namespace:=z1_gazebo sim:=false">
         <!--
     The following transforms are approximate and require further calibration.
@@ -38,8 +38,7 @@
         </link>
         <!-- add RealSense D435i (the mesh is actually the non-IMU version) -->
-        <xacro:property name="simulation" value="true" />
         <xacro:include filename="$(find realsense2_description)/urdf/_d435i.urdf.xacro" />
-        <xacro:sensor_d435i name="wrist_camera" parent="z1_realsense_mount"
-            use_nominal_extrinsics="${simulation}">
+        <xacro:sensor_d435i name="${robot_namespace}/wrist_camera" parent="z1_realsense_mount"
+            use_nominal_extrinsics="${sim}">
             <origin xyz="0.008 0.0 0.0375" rpy="0.0 0.0 0.0" /> <!-- screw holes line up, but may
             need further calibration -->
@@ -49,5 +48,5 @@
             filename="$(find z1_description)/xacro/realsense_d435.gazebo" />
         <!-- Add front camera -->
-        <xacro:realsense_d435_gazebo name="wrist_camera">
+        <xacro:realsense_d435_gazebo name="${robot_namespace}/wrist_camera">
             <origin xyz="0 0 0" rpy="0 0 0" />
         </xacro:realsense_d435_gazebo>

Commit message: Add rotational offset to robotiq gripper to match real arm

File: robots/z1_description/xacro/z1.xacro (robot description, xacro)
@@ -313,5 +313,5 @@
                 <visual>
                     <!-- Approximate -->
-                    <origin xyz="0 0 0" rpy="0 0 0.4" />
+                    <origin xyz="0 0 0" rpy="0 0 ${22.5*2*pi/360}" />
                     <geometry>
                         <mesh
@@ -331,5 +331,6 @@
             </link>
             <joint name="link6_to_adapter_sleeve" type="fixed">
-                <origin xyz="0.044 0 0" rpy="${pi/2} 0 -${pi/2}" />
+                <origin xyz="0.044 0 0" rpy="${pi/2} -${22.5*2*pi/360} -${pi/2}" /> <!-- 22.5 degree
+                rotational offset to match real arm -->
                 <parent link="link06" />
                 <child link="Adapter_Sleeve_Robotiq" />

Commit message: Added spacer for robotiq gripper

File: robots/z1_description/xacro/z1.xacro (robot description, xacro)
@@ -310,5 +310,5 @@
         </xacro:if>
         <xacro:if value="${robotiq_gripper}">
-            <link name="Adapter_Sleeve_Robotiq">
+            <link name="adapter_sleeve_robotiq">
                 <visual>
                     <!-- Approximate -->
@@ -326,5 +326,5 @@
                     <origin xyz="0 0 ${-0.02/2}" rpy="0 0 0" />
                     <geometry>
-                        <cylinder length="0.02" radius="0.045" />
+                        <cylinder length="0.02" radius="0.0445" />
                     </geometry>
                 </collision>
@@ -334,16 +334,52 @@
                 rotational offset to match real arm -->
                 <parent link="link06" />
-                <child link="Adapter_Sleeve_Robotiq" />
-            </joint>
-            <gazebo reference="Adapter_Sleeve_Robotiq">
+                <child link="adapter_sleeve_robotiq" />
+            </joint>
+            <gazebo reference="adapter_sleeve_robotiq">
                 <material>Gazebo/Grey</material>
             </gazebo>
+            <joint name="adapter_sleeve_to_wrist_spacer" type="fixed">
+                <origin xyz="0 0 -0.0202" rpy="0 0 0" />
+                <parent link="adapter_sleeve_robotiq" />
+                <child link="robotiq_wrist_spacer" />
+            </joint>
+            <xacro:property name="spacer_length" value="0.015" />
+            <!-- Robotiq Wrist Spacer -->
+            <link name="robotiq_wrist_spacer">
+                <visual>
+                    <origin xyz="0 0 -${spacer_length/2}" rpy="0 0 0" />
+                    <geometry>
+                        <cylinder length="${spacer_length}" radius="0.0445" />
+                    </geometry>
+                    <material name="black">
+                        <color rgba="${0/255} ${0/255} ${0/255} 1" />
+                    </material>
+                </visual>
+                <collision>
+                    <origin xyz="0 0 -${spacer_length/2}" rpy="0 0 0" />
+                    <geometry>
+                        <cylinder length="${spacer_length}" radius="0.045" />
+                    </geometry>
+                </collision>
+            </link>
             <!-- Robotiq Force Torque FT 300-->
             <xacro:include filename="$(find robotiq_ft_sensor)/urdf/robotiq_ft300.urdf.xacro" />
-            <xacro:robotiq_ft300 parent="Adapter_Sleeve_Robotiq" prefix=""
+            <xacro:robotiq_ft300 parent="robotiq_wrist_spacer" prefix=""
                 gazebo="${sim}" ft_topic="${robot_namespace}/robotiq_ft_wrench">
                 <!-- XYZ NEEDS TUNING -->
-                <origin xyz="0 0 -0.02" rpy="${pi} 0 -${pi/2}" />
+                <origin xyz="0 0 ${-spacer_length+0.004}" rpy="${pi} 0 -${pi/2}" />
             </xacro:robotiq_ft300>
+            <!-- <link name="test" />
+            <joint name="test_joint" type="fixed">
+                <parent link="adapter_sleeve_robotiq" />
+                <child link="test" />
+                <origin xyz="0 0 -0.163" rpy="0 0 0" />
+            </joint>
+            <link name="test2" />
+            <joint name="test2_joint" type="fixed">
+                <parent link="test" />
+                <child link="test2" />
+                <origin xyz="0 0.03 0" rpy="0 0 0" />
+            </joint> -->
             <!-- Robotiq 2F140 -->
             <xacro:include
@@ -390,5 +426,5 @@
                     use_nominal_extrinsics="${sim}">
                     <!-- XYZ NEEDS TUNING -->
-                    <origin xyz="0.02 0 0.0465" rpy="${pi} -${pi/2} 0" />
+                    <origin xyz="0.018 0 0.049" rpy="${pi} -${pi/2} 0" />
                 </xacro:sensor_d435i>
                 <!-- Simulated Realsense -->
