Commit message: Rewrite Z1 xacro as macro, add realsense mount option, add robotiq gripper option

File: robots/z1_description/xacro/const.xacro (robot description, xacro)
@@ -70,5 +70,5 @@
     <xacro:property name="L05_Izz" value="0.00053860"/>
     <!-- Link 06 -->
-    <xacro:property name="L06_Mass" value="0.28875807"/>
+    <!-- <xacro:property name="L06_Mass" value="0.28875807"/>
     <xacro:property name="L06_ComX" value="0.02415690"/>
     <xacro:property name="L06_ComY" value="-0.00017355"/>
@@ -79,7 +79,18 @@
     <xacro:property name="L06_Iyy" value="0.00014750"/>
     <xacro:property name="L06_Iyz" value="0.00000008"/>
-    <xacro:property name="L06_Izz" value="0.00014680"/>
+    <xacro:property name="L06_Izz" value="0.00014680"/> -->
+    <!-- Increased intertias for sim stability -->
+    <xacro:property name="L06_Mass" value="0.28875807"/>
+    <xacro:property name="L06_ComX" value="0.02415690"/>
+    <xacro:property name="L06_ComY" value="-0.00017355"/>
+    <xacro:property name="L06_ComZ" value="-0.00143876"/>
+    <xacro:property name="L06_Ixx" value="0.0009"/>
+    <xacro:property name="L06_Ixy" value="0.000006"/>
+    <xacro:property name="L06_Ixz" value="0.0000027"/>
+    <xacro:property name="L06_Iyy" value="0.00075"/>
+    <xacro:property name="L06_Iyz" value="0.0000004"/>
+    <xacro:property name="L06_Izz" value="0.00075"/>
     <!-- Link Gripper Stator -->
-    <xacro:property name="GripperStator_Mass" value="0.52603655"/>
+    <!-- <xacro:property name="GripperStator_Mass" value="0.52603655"/>
     <xacro:property name="GripperStator_ComX" value="0.04764427"/>
     <xacro:property name="GripperStator_ComY" value="-0.00035819"/>
@@ -90,7 +101,18 @@
     <xacro:property name="GripperStator_Iyy" value="0.00068614"/>
     <xacro:property name="GripperStator_Iyz" value="0.00000209"/>
-    <xacro:property name="GripperStator_Izz" value="0.00066293"/>
+    <xacro:property name="GripperStator_Izz" value="0.00066293"/> -->
+    <!-- Increased intertias for sim stability -->
+    <xacro:property name="GripperStator_Mass" value="0.52603655"/>
+    <xacro:property name="GripperStator_ComX" value="0.04764427"/>
+    <xacro:property name="GripperStator_ComY" value="-0.00035819"/>
+    <xacro:property name="GripperStator_ComZ" value="-0.00249162"/>
+    <xacro:property name="GripperStator_Ixx" value="0.0038683"/>
+    <xacro:property name="GripperStator_Ixy" value="-0.0000359"/>
+    <xacro:property name="GripperStator_Ixz" value="0.0007662"/>
+    <xacro:property name="GripperStator_Iyy" value="0.0068614"/>
+    <xacro:property name="GripperStator_Iyz" value="0.0000209"/>
+    <xacro:property name="GripperStator_Izz" value="0.0066293"/>
     <!-- Link Gripper Mover -->
-    <xacro:property name="GripperMover_Mass" value="0.27621302"/>
+    <!-- <xacro:property name="GripperMover_Mass" value="0.27621302"/>
     <xacro:property name="GripperMover_ComX" value="0.01320633"/>
     <xacro:property name="GripperMover_ComY" value="0.00476708"/>
@@ -101,5 +123,16 @@
     <xacro:property name="GripperMover_Iyy" value="0.00026787"/>
     <xacro:property name="GripperMover_Iyz" value="0.00000262"/>
-    <xacro:property name="GripperMover_Izz" value="0.00035728"/>
+    <xacro:property name="GripperMover_Izz" value="0.00035728"/> -->
+    <!-- Increased intertias for sim stability -->
+    <xacro:property name="GripperMover_Mass" value="0.27621302"/>
+    <xacro:property name="GripperMover_ComX" value="0.01320633"/>
+    <xacro:property name="GripperMover_ComY" value="0.00476708"/>
+    <xacro:property name="GripperMover_ComZ" value="0.00380534"/>
+    <xacro:property name="GripperMover_Ixx" value="0.0017716"/>
+    <xacro:property name="GripperMover_Ixy" value="0.0001683"/>
+    <xacro:property name="GripperMover_Ixz" value="-0.0001786"/>
+    <xacro:property name="GripperMover_Iyy" value="0.0026787"/>
+    <xacro:property name="GripperMover_Iyz" value="0.0000262"/>
+    <xacro:property name="GripperMover_Izz" value="0.0035728"/>
     <!-- joint limits -->
     <xacro:property name="jointDamping" value="1.0"/>

File: robots/z1_description/xacro/gazebo.xacro (robot description, xacro)
@@ -14,5 +14,5 @@
     </gazebo>
     <gazebo reference="link06">
-        <self_collide>true</self_collide>
+        <self_collide>false</self_collide>
     </gazebo>
 </robot>

Commit message: Reverted Z1 inertias for link06 and gripperStator (change back to modded values if gazebo crashes), added end_effector link for unitree gripper

File: robots/z1_description/xacro/const.xacro (robot description, xacro)
@@ -70,5 +70,5 @@
     <xacro:property name="L05_Izz" value="0.00053860"/>
     <!-- Link 06 -->
-    <!-- <xacro:property name="L06_Mass" value="0.28875807"/>
+    <xacro:property name="L06_Mass" value="0.28875807"/>
     <xacro:property name="L06_ComX" value="0.02415690"/>
     <xacro:property name="L06_ComY" value="-0.00017355"/>
@@ -79,7 +79,7 @@
     <xacro:property name="L06_Iyy" value="0.00014750"/>
     <xacro:property name="L06_Iyz" value="0.00000008"/>
-    <xacro:property name="L06_Izz" value="0.00014680"/> -->
+    <xacro:property name="L06_Izz" value="0.00014680"/>
     <!-- Increased intertias for sim stability -->
-    <xacro:property name="L06_Mass" value="0.28875807"/>
+    <!-- <xacro:property name="L06_Mass" value="0.28875807"/>
     <xacro:property name="L06_ComX" value="0.02415690"/>
     <xacro:property name="L06_ComY" value="-0.00017355"/>
@@ -90,7 +90,7 @@
     <xacro:property name="L06_Iyy" value="0.00075"/>
     <xacro:property name="L06_Iyz" value="0.0000004"/>
-    <xacro:property name="L06_Izz" value="0.00075"/>
+    <xacro:property name="L06_Izz" value="0.00075"/> -->
     <!-- Link Gripper Stator -->
-    <!-- <xacro:property name="GripperStator_Mass" value="0.52603655"/>
+    <xacro:property name="GripperStator_Mass" value="0.52603655"/>
     <xacro:property name="GripperStator_ComX" value="0.04764427"/>
     <xacro:property name="GripperStator_ComY" value="-0.00035819"/>
@@ -101,7 +101,7 @@
     <xacro:property name="GripperStator_Iyy" value="0.00068614"/>
     <xacro:property name="GripperStator_Iyz" value="0.00000209"/>
-    <xacro:property name="GripperStator_Izz" value="0.00066293"/> -->
+    <xacro:property name="GripperStator_Izz" value="0.00066293"/>
     <!-- Increased intertias for sim stability -->
-    <xacro:property name="GripperStator_Mass" value="0.52603655"/>
+    <!-- <xacro:property name="GripperStator_Mass" value="0.52603655"/>
     <xacro:property name="GripperStator_ComX" value="0.04764427"/>
     <xacro:property name="GripperStator_ComY" value="-0.00035819"/>
@@ -112,5 +112,5 @@
     <xacro:property name="GripperStator_Iyy" value="0.0068614"/>
     <xacro:property name="GripperStator_Iyz" value="0.0000209"/>
-    <xacro:property name="GripperStator_Izz" value="0.0066293"/>
+    <xacro:property name="GripperStator_Izz" value="0.0066293"/> -->
     <!-- Link Gripper Mover -->
     <!-- <xacro:property name="GripperMover_Mass" value="0.27621302"/>

File: robots/z1_description/xacro/z1.xacro (robot description, xacro)
@@ -308,4 +308,11 @@
                 <xacro:z1_realsense_wrist_mount robot_namespace="${robot_namespace}" sim="${sim}" />
             </xacro:if>
+            <!-- End-effector link to match unitree gripper convention (x-axis forward) -->
+            <link name="end_effector" />
+            <joint name="gripper_to_end_effector" type="fixed">
+                <origin xyz="0.135 0 0" rpy="0 0 0" />
+                <parent link="gripperStator" />
+                <child link="end_effector" />
+            </joint>
         </xacro:if>
         <xacro:if value="${robotiq_gripper}">
